File: Illuminator.kicad_pcb (KiCad board)
At the start: 2 copper layers, 17 parts, among them J0 Conn_01x03_Male, Q0 DMG1012UW

Commit message: Applying script
Parts:
- J0, Q0: moved to B.Cu
- moved LED6 82.0 mm to (90.2, 128.3), turned to 160.948 degrees
- moved LED5 77.5 mm to (71.7, 109.7), turned to 108.812 degrees
- moved LED3 70.3 mm to (82.1, 76.0), turned to 36.8121 degrees
- moved LED4 67.7 mm to (70.1, 99.5), turned to 88.948 degrees
- moved R2 67.4 mm to (71.8, 89.8), turned to 250.136 degrees
- moved R4 64.3 mm to (116.8, 124.8), turned to 34.1359 degrees
- moved R3 62.6 mm to (81.6, 123.7), turned to 322.136 degrees
- moved Q0 57.1 mm to (72.1, 100.0)
- moved LED7 54.7 mm to (100.4, 129.9), turned to 180.812 degrees
- moved LED2 52.3 mm to (91.3, 71.4), turned to 16.948 degrees
- moved R1 48.3 mm to (101.0, 70.0), turned to 178.136 degrees
- moved LED8 41.1 mm to (123.9, 118.0), turned to 232.948 degrees
- moved LED9 28.8 mm to (128.6, 108.8), turned to 252.812 degrees
- moved LED1 27.4 mm to (117.3, 75.5), turned to 324.812 degrees
- moved LED0 18.2 mm to (124.5, 82.8), turned to 304.948 degrees
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Routing:
- net /TO_5V: track 0.00 -> 248.6 mm, vias 0 -> 1
- net Net-(LED1-Pad1): track 0.00 -> 210.5 mm, vias 0 -> 1
- net /TO_GND: track 0.00 -> 89.9 mm
- net /TO_3V3: track 0.00 -> 89.9 mm
- net Net-(LED2-Pad1): track 0.00 -> 6.60 mm
- net Net-(LED0-Pad1): track 0.00 -> 6.60 mm
- net Net-(LED6-Pad1): track 0.00 -> 6.60 mm
- net Net-(LED2-Pad2): track 0.00 -> 6.60 mm
- net Net-(LED4-Pad2): track 0.00 -> 6.60 mm
- net Net-(LED0-Pad2): track 0.00 -> 6.60 mm
- net Net-(LED8-Pad2): track 0.00 -> 6.60 mm
- net Net-(LED6-Pad2): track 0.00 -> 6.60 mm
- net Net-(LED8-Pad1): track 0.00 -> 6.60 mm
- net Net-(LED4-Pad1): track 0.00 -> 6.60 mm
- added copper zone on F.Cu, net /TO_5V
- added copper zone on F.Cu, net Net-(LED0-Pad1)
- added copper zone on F.Cu, net Net-(LED0-Pad2)
- added copper zone on F.Cu, net Net-(LED1-Pad1)
- added copper zone on F.Cu, net Net-(LED2-Pad1)
- added copper zone on F.Cu, net Net-(LED2-Pad2)
- added copper zone on F.Cu, net Net-(LED4-Pad1)
- added copper zone on F.Cu, net Net-(LED4-Pad2)
- added copper zone on F.Cu, net Net-(LED6-Pad1)
- added copper zone on F.Cu, net Net-(LED6-Pad2)
- added copper zone on F.Cu, net Net-(LED8-Pad1)
- added copper zone on F.Cu, net Net-(LED8-Pad2)
