File: Illuminator.kicad_pcb (KiCad board)
At the start: 2 copper layers, 58.5 x 58.5 mm, 33 parts, among them J0 Conn_02x03_Top_Bottom, Q0 DMG1012UW, U1 VEML7700

Commit message: Cleaning up schematics and remapping all elements in the PCB to the new netlist.
Parts:
- GND, LED: value Measurement_Point_Round-SMD-Pad_Small -> Test_Point
- turned C0 to 270 degrees
- turned R_PU1 to 180 degrees
- turned R_PU2 to 180 degrees
Connections:
- net /TO_5V renamed +5V
- C0 pad 1: /TO_GND -> +3V3
- C0 pad 2: /TO_3V3 -> GND
- GND pad 1: /TO_GND -> GND
- J0 pad 3: /TO_GND -> GND
- J0 pad 4: /TO_3V3 -> +3V3
- Q0 pad 2: /TO_GND -> GND
- R_PU1 pad 1: /TO_3V3 -> /TO_SCL
- R_PU1 pad 2: /TO_SCL -> +3V3
- R_PU2 pad 1: /TO_3V3 -> /TO_SDA
- R_PU2 pad 2: /TO_SDA -> +3V3
- U1 pad 2: /TO_3V3 -> +3V3
- U1 pad 3: /TO_GND -> GND
Routing:
- net /TO_3V3: track 27.5 -> 0.00 mm, vias 1 -> 0
- net +3V3: track 0.00 -> 27.5 mm, vias 0 -> 1
- net GND: vias 0 -> 1
- net /TO_GND: vias 1 -> 0
- added copper zone on B.Cu, net GND
- added copper zone on F.Cu, net GND
- removed copper zone on B.Cu, net /TO_GND
- removed copper zone on F.Cu, net /TO_GND

Commit message: Saved export settings
Other:
- board text added: "Ratcam Illuminator http://bit.ly/2m9yLHR"
- board text removed: "http://bit.ly/2m9yLHR"
Changed lines of the file:
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@@
   (layers
     (0 F.Cu signal)
-    (31 B.Cu signal hide)
+    (31 B.Cu signal)
     (32 B.Adhes user)
     (33 F.Adhes user)
@@
     (aux_axis_origin 0 0)
     (grid_origin 100 100)
-    (visible_elements FFFEFF7F)
+    (visible_elements FFFFFF7F)
     (pcbplotparams
-      (layerselection 0x010fc_ffffffff)
-      (usegerberextensions false)
+      (layerselection 0x010f0_ffffffff)
+      (usegerberextensions true)
       (usegerberattributes false)
       (usegerberadvancedattributes false)
@@
       (psa4output false)
       (plotreference true)
-      (plotvalue true)
+      (plotvalue false)
       (plotinvisibletext false)
       (padsonsilk false)
-      (subtractmaskfromsilk false)
+      (subtractmaskfromsilk true)
       (outputformat 1)
       (mirror false)
-      (drillshape 1)
+      (drillshape 0)
       (scaleselection 1)
-      (outputdirectory ""))
+      (outputdirectory Export/Mark1/))
   )
   (net 0 "")
@@
       (effects (font (size 1 1) (thickness 0.15)) (justify mirror))
     )
-    (fp_text value "Ratcam Illuminator" (at 0 3.175) (layer F.SilkS)
-      (effects (font (size 1 1) (thickness 0.15)))
+    (fp_text value "Ratcam Illuminator" (at 0 6.35) (layer B.SilkS) hide
+      (effects (font (size 1 1) (thickness 0.15)) (justify mirror))
     )
     (fp_poly (pts (xy 4.906667 -4.906667) (xy 5.333333 -4.906667) (xy 5.333333 -5.333333) (xy 4.906667 -5.333333)
@@
       (xy 3.844506 1.909749)) (layer B.SilkS) (width 0.058059))
   )
-  (gr_text http://bit.ly/2m9yLHR (at 100 82.855) (layer F.SilkS)
+  (gr_text "Ratcam Illuminator\nhttp://bit.ly/2m9yLHR" (at 100 81.966) (layer F.SilkS)
     (effects (font (size 1 1) (thickness 0.15)))
   )
